Commit message: given input error

File: urdf/my_robot_x.urdf.xacro (robot description, xacro)
@@ -31,4 +31,10 @@
     </xacro:macro>
     <!-- LINK LIST -->
+    <link name="map">
+    </link>
+    <joint name="map_joint" type="fixed">
+        <parent link="map"/>
+        <child link="base_link"/>
+    </joint>
     <!--Body/Chassis of the robot-->
     <link name="base_link">
@@ -111,5 +117,5 @@
         <topicName>ground_truth/state</topicName>
         <gaussianNoise>0.01</gaussianNoise>
-        <frameName>base_link</frameName>
+        <frameName>map</frameName>
         <xyzOffsets>0 0 0</xyzOffsets>
         <rpyOffsets>0 0 0</rpyOffsets>
