Commit message: Implement eight in nonLinear control

File: urdf/cylinder_wheel.urdf.xacro (robot description, xacro)
@@ -48,5 +48,5 @@
       <origin xyz="${translateX * base_x_origin_to_wheel_origin} ${translateY * base_y_origin_to_wheel_origin} ${base_z_origin_to_wheel_origin}" rpy="0 0 0" />
       <axis xyz="0 1 0" rpy="0  0" />
-      <limit effort="100" velocity="100"/>
+      <limit effort="100" velocity="50"/>
       <joint_properties damping="0.0" friction="0.0"/>
     </joint>
